Commit message: [feat] support multi-robot profile in autosim pipeline.

File: lw_benchhub/autosim/content/assets/robot/x7s/urdf/X7S.urdf (robot description, URDF)
Before this commit: robot X7S, 29 links, 28 joints
Joints:
- removed joint base_yaw_joint
- added joint base_yaw_link: type revolute, parent base_y_link, child base_yaw_link, origin xyz=0 0 0 rpy=0 0 0, axis 0 0 1, limit lower=-6.28159 upper=6.28159 effort=100 velocity=1000
