Commit message: complete open fridge.

File: lw_benchhub/autosim/content/assets/robot/g1/urdf/G1.urdf (robot description, URDF)
Before this commit: robot g1_autosim, 57 links, 56 joints
Links:
- added link left_g1_loco_ee_tip, mass 0.001
Joints:
- added joint left_g1_loco_ee_tip_fixed: type fixed, parent left_hand_palm_link, child left_g1_loco_ee_tip, origin xyz=0.1235 0.0016 -0.0285 rpy=0 0 0
